Commit message: optimization witih pythod

File: src/drake_opt/franka_description/urdf/panda.urdf (robot description, URDF)
Before this commit: robot panda, 12 links, 11 joints
Links:
- removed link panda_link8
- link panda_hand: geometry collision mesh filename=../meshes/visual/hand_simple.obj; visual mesh filename=../meshes/visual/hand.obj
- link panda_leftfinger: geometry collision mesh filename=../meshes/visual/finger_simple.obj; visual mesh filename=../meshes/visual/finger.obj
- link panda_link0: geometry collision mesh filename=../meshes/visual/link0_simple.obj; visual mesh filename=../meshes/visual/link0.obj
- link panda_link1: geometry collision mesh filename=../meshes/visual/link1_simple.obj; visual mesh filename=../meshes/visual/link1.obj
- link panda_link2: geometry collision mesh filename=../meshes/visual/link2_simple.obj; visual mesh filename=../meshes/visual/link2.obj
- link panda_link3: geometry collision mesh filename=../meshes/visual/link3_simple.obj; visual mesh filename=../meshes/visual/link3.obj
- link panda_link4: geometry collision mesh filename=../meshes/visual/link4_simple.obj; visual mesh filename=../meshes/visual/link4.obj
- link panda_link5: geometry collision mesh filename=../meshes/visual/link5_simple.obj; visual mesh filename=../meshes/visual/link5.obj
- link panda_link6: geometry collision mesh filename=../meshes/visual/link6_simple.obj; visual mesh filename=../meshes/visual/link6.obj
- link panda_link7: geometry collision mesh filename=../meshes/visual/link7_simple.obj; visual mesh filename=../meshes/visual/link7.obj
- link panda_rightfinger: geometry collision mesh filename=../meshes/visual/finger_simple.obj; visual mesh filename=../meshes/visual/finger.obj
Joints:
- removed joint panda_joint8
- joint panda_hand_joint: origin xyz=0 0 0 rpy=0 0 -0.785398163397 -> xyz=0 0 0.107 rpy=0 0 -0.785398163397; parent panda_link8 -> panda_link7
